Commit message: Update turtlebot3_burger.urdf
屁眼

File: src/summer_robot/urdf/turtlebot3_burger.urdf (robot description, URDF)
Before this commit: robot turtlebot3_burger, 8 links, 7 joints
Joints:
- joint ${namespace}camera_joint: origin xyz=0.04 0 0.13 rpy=0 0.785 0 -> xyz=0.04 0 0.13 rpy=0 0 0

Commit message: Enhance exploration logic, tune params, and disable ground scanner
- URDF: Change camera to a downward-facing wide-angle camera.
- Launch: Temporarily disable ground_scanner_launch to isolate navigation testing.
- Params: Increase decision_rate to 2.0 Hz, sync Nav2 inflation_radius with explorer to 0.25.
- algorithms.py: Increase stickiness bonus to prevent target oscillation, penalize backward turning.
- controller.py: Add distance check to send_goal to avoid interrupting same target. Fix Action Client preemption bug to correctly ignore aborted old goals.
- explorer_node.py: Fix Watchdog logic and early returns. Lock navigation target during traversal, relying on Nav2's built-in progress checker. Decrease dynamic blacklist radius to prevent masking the whole map.

File: src/summer_robot/urdf/turtlebot3_burger.urdf (robot description, URDF)
Before this commit: robot turtlebot3_burger, 8 links, 7 joints
Joints:
- joint ${namespace}camera_joint: origin xyz=0.04 0 0.13 rpy=0 0 0 -> xyz=0.10 0 0.13 rpy=0 1.5708 0
